Commit message: Update VICA description

File: src/vica_description/urdf/VICA.xacro (robot description, xacro)
@@ -17,7 +17,7 @@
 <link name="base_link">
   <inertial>
-    <origin xyz="0.30817684998290357 0.0 0.2398462811293035" rpy="0 0 0"/>
-    <mass value="100.3733798045696"/>
-    <inertia ixx="2.797826" iyy="4.141308" izz="4.614014" ixy="-0.0" iyz="0.0" ixz="0.369915"/>
+    <origin xyz="0.004031215194176557 3.002726997808124e-17 0.07606562657816282" rpy="0 0 0"/>
+    <mass value="90.84709962539795"/>
+    <inertia ixx="2.402108" iyy="3.622523" izz="4.166828" ixy="0.0" iyz="-0.0" ixz="0.343284"/>
   </inertial>
   <visual>
@@ -37,10 +37,10 @@
 <link name="left_wheel_1">
   <inertial>
-    <origin xyz="2.1094237467877974e-15 0.035687655502016025 1.3877787807814457e-17" rpy="0 0 0"/>
+    <origin xyz="2.0539125955565396e-15 0.03668765550201605 0.0" rpy="0 0 0"/>
     <mass value="0.5663250710944822"/>
     <inertia ixx="0.000634" iyy="0.001025" izz="0.000634" ixy="0.0" iyz="-0.0" ixz="0.0"/>
   </inertial>
   <visual>
-    <origin xyz="-0.459 -0.1465 -0.065" rpy="0 0 0"/>
+    <origin xyz="-0.154 -0.1465 0.084" rpy="0 0 0"/>
     <geometry>
       <mesh filename="package://vica_description/meshes/left_wheel_1.stl" scale="0.001 0.001 0.001"/>
@@ -49,5 +49,5 @@
   </visual>
   <collision>
-    <origin xyz="-0.459 -0.1465 -0.065" rpy="0 0 0"/>
+    <origin xyz="-0.154 -0.1465 0.084" rpy="0 0 0"/>
     <geometry>
       <mesh filename="package://vica_description/meshes/left_wheel_1.stl" scale="0.001 0.001 0.001"/>
@@ -57,10 +57,10 @@
 <link name="right_wheel_1">
   <inertial>
-    <origin xyz="-3.447242491461111e-14 -0.03568765550201608 0.0" rpy="0 0 0"/>
+    <origin xyz="-0.00046568184733652984 -0.03568765550201608 0.0009570426748952837" rpy="0 0 0"/>
     <mass value="0.5663250710944814"/>
-    <inertia ixx="0.000634" iyy="0.001025" izz="0.000634" ixy="-0.0" iyz="-0.0" ixz="0.0"/>
-  </inertial>
-  <visual>
-    <origin xyz="-0.459 0.1465 -0.065" rpy="0 0 0"/>
+    <inertia ixx="0.000634" iyy="0.001025" izz="0.000634" ixy="0.0" iyz="0.0" ixz="-0.0"/>
+  </inertial>
+  <visual>
+    <origin xyz="-0.154 0.1465 0.084" rpy="0 0 0"/>
     <geometry>
       <mesh filename="package://vica_description/meshes/right_wheel_1.stl" scale="0.001 0.001 0.001"/>
@@ -69,5 +69,5 @@
   </visual>
   <collision>
-    <origin xyz="-0.459 0.1465 -0.065" rpy="0 0 0"/>
+    <origin xyz="-0.154 0.1465 0.084" rpy="0 0 0"/>
     <geometry>
       <mesh filename="package://vica_description/meshes/right_wheel_1.stl" scale="0.001 0.001 0.001"/>
@@ -77,10 +77,10 @@
 <link name="front_left_caster_wheel_1">
   <inertial>
-    <origin xyz="-1.6792123247455493e-15 0.01574568542726719 2.7755575615628914e-17" rpy="0 0 0"/>
+    <origin xyz="-1.6653345369377348e-15 0.01574568542726719 0.0" rpy="0 0 0"/>
     <mass value="0.11451893837110633"/>
     <inertia ixx="4.7e-05" iyy="7.8e-05" izz="4.7e-05" ixy="-0.0" iyz="0.0" ixz="0.0"/>
   </inertial>
   <visual>
-    <origin xyz="-0.053 -0.0695 -0.042" rpy="0 0 0"/>
+    <origin xyz="0.252 -0.0695 0.107" rpy="0 0 0"/>
     <geometry>
       <mesh filename="package://vica_description/meshes/front_left_caster_wheel_1.stl" scale="0.001 0.001 0.001"/>
@@ -89,5 +89,5 @@
   </visual>
   <collision>
-    <origin xyz="-0.053 -0.0695 -0.042" rpy="0 0 0"/>
+    <origin xyz="0.252 -0.0695 0.107" rpy="0 0 0"/>
     <geometry>
       <mesh filename="package://vica_description/meshes/front_left_caster_wheel_1.stl" scale="0.001 0.001 0.001"/>
@@ -97,10 +97,10 @@
 <link name="front_right_caster_wheel_1">
   <inertial>
-    <origin xyz="5.169475958410885e-15 -0.015745685427267203 1.3877787807814457e-17" rpy="0 0 0"/>
+    <origin xyz="5.162537064506978e-15 -0.015745685427267203 0.0" rpy="0 0 0"/>
     <mass value="0.11451893837110629"/>
-    <inertia ixx="4.7e-05" iyy="7.8e-05" izz="4.7e-05" ixy="-0.0" iyz="0.0" ixz="0.0"/>
-  </inertial>
-  <visual>
-    <origin xyz="-0.053 0.0695 -0.042" rpy="0 0 0"/>
+    <inertia ixx="4.7e-05" iyy="7.8e-05" izz="4.7e-05" ixy="-0.0" iyz="0.0" ixz="-0.0"/>
+  </inertial>
+  <visual>
+    <origin xyz="0.252 0.0695 0.107" rpy="0 0 0"/>
     <geometry>
       <mesh filename="package://vica_description/meshes/front_right_caster_wheel_1.stl" scale="0.001 0.001 0.001"/>
@@ -109,5 +109,5 @@
   </visual>
   <collision>
-    <origin xyz="-0.053 0.0695 -0.042" rpy="0 0 0"/>
+    <origin xyz="0.252 0.0695 0.107" rpy="0 0 0"/>
     <geometry>
       <mesh filename="package://vica_description/meshes/front_right_caster_wheel_1.stl" scale="0.001 0.001 0.001"/>
@@ -117,10 +117,10 @@
 <link name="front_right_caster_steer_1">
   <inertial>
-    <origin xyz="-0.00408089404459451 0.0037449849629774684 -0.01766662210223026" rpy="0 0 0"/>
+    <origin xyz="-0.004080894044594496 0.0037449849629774684 -0.017666622102230287" rpy="0 0 0"/>
     <mass value="0.9536308497491053"/>
     <inertia ixx="0.000637" iyy="0.000626" izz="0.000908" ixy="4e-05" iyz="8.5e-05" ixz="-8.2e-05"/>
   </inertial>
   <visual>
-    <origin xyz="-0.083 0.0845 -0.1075" rpy="0 0 0"/>
+    <origin xyz="0.222 0.0845 0.0415" rpy="0 0 0"/>
     <geometry>
       <mesh filename="package://vica_description/meshes/front_right_caster_steer_1.stl" scale="0.001 0.001 0.001"/>
@@ -129,5 +129,5 @@
   </visual>
   <collision>
-    <origin xyz="-0.083 0.0845 -0.1075" rpy="0 0 0"/>
+    <origin xyz="0.222 0.0845 0.0415" rpy="0 0 0"/>
     <geometry>
       <mesh filename="package://vica_description/meshes/front_right_caster_steer_1.stl" scale="0.001 0.001 0.001"/>
@@ -137,10 +137,10 @@
 <link name="front_left_caster_steer_1">
   <inertial>
-    <origin xyz="-0.00408089404459451 -0.003744984962977496 -0.01766662210223026" rpy="0 0 0"/>
+    <origin xyz="-0.004080894044594496 -0.003744984962977496 -0.017666622102230287" rpy="0 0 0"/>
     <mass value="0.9536308497491053"/>
     <inertia ixx="0.000637" iyy="0.000626" izz="0.000908" ixy="-4e-05" iyz="-8.5e-05" ixz="-8.2e-05"/>
   </inertial>
   <visual>
-    <origin xyz="-0.083 -0.0845 -0.1075" rpy="0 0 0"/>
+    <origin xyz="0.222 -0.0845 0.0415" rpy="0 0 0"/>
     <geometry>
       <mesh filename="package://vica_description/meshes/front_left_caster_steer_1.stl" scale="0.001 0.001 0.001"/>
@@ -149,5 +149,5 @@
   </visual>
   <collision>
-    <origin xyz="-0.083 -0.0845 -0.1075" rpy="0 0 0"/>
+    <origin xyz="0.222 -0.0845 0.0415" rpy="0 0 0"/>
     <geometry>
       <mesh filename="package://vica_description/meshes/front_left_caster_steer_1.stl" scale="0.001 0.001 0.001"/>
@@ -157,10 +157,10 @@
 <link name="laser_frame">
   <inertial>
-    <origin xyz="0.0 0.0 0.010868727234877307" rpy="0 0 0"/>
+    <origin xyz="0.0 0.0 0.010868727234877334" rpy="0 0 0"/>
     <mass value="0.16353480730457975"/>
     <inertia ixx="5.9e-05" iyy="5.9e-05" izz="0.000105" ixy="0.0" iyz="-0.0" ixz="-0.0"/>
   </inertial>
   <visual>
-    <origin xyz="-${laser_x} -${laser_y} -${laser_z}" rpy="0 0 0"/>
+    <origin xyz="-0.185 -0.0 -0.236" rpy="0 0 0"/>
     <geometry>
       <mesh filename="package://vica_description/meshes/lidar_1.stl" scale="0.001 0.001 0.001"/>
@@ -169,5 +169,5 @@
   </visual>
   <collision>
-    <origin xyz="-${laser_x} -${laser_y} -${laser_z}" rpy="0 0 0"/>
+    <origin xyz="-0.185 -0.0 -0.236" rpy="0 0 0"/>
     <geometry>
       <mesh filename="package://vica_description/meshes/lidar_1.stl" scale="0.001 0.001 0.001"/>
@@ -177,5 +177,5 @@
 <link name="camera_link"/>
 <joint name="left_wheel_joint" type="continuous">
-  <origin xyz="0.459 0.1465 0.065" rpy="0 0 0"/>
+  <origin xyz="0.154 0.1465 -0.084" rpy="0 0 0"/>
   <parent link="base_link"/>
   <child link="left_wheel_1"/>
@@ -183,5 +183,5 @@
 </joint>
 <joint name="right_wheel_joint" type="continuous">
-  <origin xyz="0.459 -0.1465 0.065" rpy="0 0 0"/>
+  <origin xyz="0.154 -0.1465 -0.084" rpy="0 0 0"/>
   <parent link="base_link"/>
   <child link="right_wheel_1"/>
@@ -201,5 +201,5 @@
 </joint>
 <joint name="front_right_caster_steer_joint" type="continuous">
-  <origin xyz="0.083 -0.0845 0.1075" rpy="0 0 0"/>
+  <origin xyz="-0.222 -0.0845 -0.0415" rpy="0 0 0"/>
   <parent link="base_link"/>
   <child link="front_right_caster_steer_1"/>
@@ -207,5 +207,5 @@
 </joint>
 <joint name="front_left_caster_steer_joint" type="continuous">
-  <origin xyz="0.083 0.0845 0.1075" rpy="0 0 0"/>
+  <origin xyz="-0.222 0.0845 -0.0415" rpy="0 0 0"/>
   <parent link="base_link"/>
   <child link="front_left_caster_steer_1"/>
@@ -213,5 +213,5 @@
 </joint>
 <joint name="laser_joint" type="fixed">
-  <origin xyz="${laser_x} ${laser_y} ${laser_z}" rpy="0 0 0"/>
+  <origin xyz="0.185 0.0 0.236" rpy="0 0 0"/>
   <parent link="base_link"/>
   <child link="laser_frame"/>

Commit message: Update VICA description visuals and camera link

File: src/vica_description/urdf/VICA.xacro (robot description, xacro)
@@ -176,5 +176,14 @@
   </collision>
 </link>
-<link name="camera_link"/>
+<link name="camera_link">
+  <!-- D455 visual placeholder: 26 x 124 x 29 mm -->
+  <visual name="d455_body">
+    <origin xyz="0 0 0" rpy="0 0 0"/>
+    <geometry>
+      <box size="0.026 0.124 0.029"/>
+    </geometry>
+    <material name="silver"/>
+  </visual>
+</link>
 <joint name="left_wheel_joint" type="continuous">
   <origin xyz="0.154 0.1465 -0.1515" rpy="0 0 0"/>

File: src/vica_description/urdf/materials.xacro (robot description, xacro)
@@ -2,5 +2,5 @@
 <robot name="VICA" xmlns:xacro="http://www.ros.org/wiki/xacro" >
 <material name="body_blue">
-  <color rgba="0 0 0 1.0"/>
+  <color rgba="0.0 0.85 0.85 1.0"/>
 </material>
 <material name="silver">

Commit message: Align VICA base and sensor TF heights

File: src/vica_description/urdf/VICA.xacro (robot description, xacro)
@@ -2,12 +2,14 @@
 <robot name="VICA" xmlns:xacro="http://www.ros.org/wiki/xacro">
 <xacro:include filename="$(find vica_description)/urdf/materials.xacro" />
-<xacro:property name="body_center_z" value="0.0675" />
-<xacro:property name="base_link_height" value="0.2165" />
+<!-- Measured heights from the ground-aligned base_footprint. -->
+<!-- base_link=0.190, laser_frame=0.382, camera_link=0.320 [m] -->
+<xacro:property name="body_center_z" value="0.044" />
+<xacro:property name="base_link_height" value="0.19" />
 <xacro:property name="laser_x" value="0.185" />
 <xacro:property name="laser_y" value="0.0" />
-<xacro:property name="laser_z" value="0.1685" />
+<xacro:property name="laser_z" value="0.192" />
 <xacro:property name="camera_x" value="0.28683" />
 <xacro:property name="camera_y" value="0.0" />
-<xacro:property name="camera_z" value="0.1084" />
+<xacro:property name="camera_z" value="0.130" />
 <link name="base_footprint"/>
 <joint name="base_footprint_joint" type="fixed">
@@ -18,5 +20,5 @@
 <link name="base_link">
   <inertial>
-    <origin xyz="0.004031215194176557 3.002726997808124e-17 0.00856562657816282" rpy="0 0 0"/>
+    <origin xyz="0.004031215194176557 3.002726997808124e-17 0.03206562657816282" rpy="0 0 0"/>
     <mass value="90.84709962539795"/>
     <inertia ixx="2.402108" iyy="3.622523" izz="4.166828" ixy="0.0" iyz="-0.0" ixz="0.343284"/>
@@ -187,5 +189,5 @@
 </link>
 <joint name="left_wheel_joint" type="continuous">
-  <origin xyz="0.154 0.1465 -0.1515" rpy="0 0 0"/>
+  <origin xyz="0.154 0.1465 -0.125" rpy="0 0 0"/>
   <parent link="base_link"/>
   <child link="left_wheel_1"/>
@@ -193,5 +195,5 @@
 </joint>
 <joint name="right_wheel_joint" type="continuous">
-  <origin xyz="0.154 -0.1465 -0.1515" rpy="0 0 0"/>
+  <origin xyz="0.154 -0.1465 -0.125" rpy="0 0 0"/>
   <parent link="base_link"/>
   <child link="right_wheel_1"/>
@@ -211,5 +213,5 @@
 </joint>
 <joint name="front_right_caster_steer_joint" type="continuous">
-  <origin xyz="-0.222 -0.0845 -0.109" rpy="0 0 0"/>
+  <origin xyz="-0.222 -0.0845 -0.0825" rpy="0 0 0"/>
   <parent link="base_link"/>
   <child link="front_right_caster_steer_1"/>
@@ -217,5 +219,5 @@
 </joint>
 <joint name="front_left_caster_steer_joint" type="continuous">
-  <origin xyz="-0.222 0.0845 -0.109" rpy="0 0 0"/>
+  <origin xyz="-0.222 0.0845 -0.0825" rpy="0 0 0"/>
   <parent link="base_link"/>
   <child link="front_left_caster_steer_1"/>
