Commit message: fix(urdf): 구동륜·캐스터 조인트 기하를 CAD·실측에 맞춘다
구동륜 간격이 0.293으로 적혀 있었다. 줄자 실측은 0.364이고 CAD 0.3618과도 2.2 mm
안에서 맞는다. 캐스터 휠은 10 mm 안쪽, 차체·라이다 메시는 3 mm 어긋나 있었다.

wheel_base_m 0.37은 그대로 둔다. 그건 회전 시험으로 맞춘 오도메트리 보정 상수라
실측 기하와 같을 필요가 없다.

-0.044를 인용하던 주석 세 곳을 같은 커밋에서 고친다. 나눠 두면 그 사이에 거짓
주석이 남는다.

visual origin이 joint origin을 정확히 상쇄해 RViz에서는 정상으로 보였고, 오차
방향이 회전축과 같아 바퀴를 굴려도 드러나지 않았다. 실물 오도메트리는 URDF를
읽지 않으므로 주행 거동은 변하지 않는다.

Co-Authored-By: Claude Opus 5 <noreply@anthropic.com>

File: src/vica_description/urdf/VICA.xacro (robot description, xacro)
@@ -4,5 +4,5 @@
 <!-- Measured heights from the ground-aligned base_footprint. -->
 <!-- base_link=0.190, laser_frame=0.382, camera_link=0.320 [m] -->
-<xacro:property name="body_center_z" value="0.044" />
+<xacro:property name="body_center_z" value="0.041" />
 <xacro:property name="base_link_height" value="0.19" />
 <xacro:property name="laser_x" value="0.185" />
@@ -20,5 +20,5 @@
 <link name="base_link">
   <inertial>
-    <origin xyz="0.004031215194176557 3.002726997808124e-17 0.03206562657816282" rpy="0 0 0"/>
+    <origin xyz="0.004031215194176557 3.002726997808124e-17 0.03506562657816282" rpy="0 0 0"/>
     <mass value="90.84709962539795"/>
     <inertia ixx="2.402108" iyy="3.622523" izz="4.166828" ixy="0.0" iyz="-0.0" ixz="0.343284"/>
@@ -45,5 +45,5 @@
   </inertial>
   <visual>
-    <origin xyz="-0.154 -0.1465 0.084" rpy="0 0 0"/>
+    <origin xyz="-0.154 -0.182 0.084" rpy="0 0 0"/>
     <geometry>
       <mesh filename="package://vica_description/meshes/left_wheel_1.stl" scale="0.001 0.001 0.001"/>
@@ -52,5 +52,5 @@
   </visual>
   <collision>
-    <origin xyz="-0.154 -0.1465 0.084" rpy="0 0 0"/>
+    <origin xyz="-0.154 -0.182 0.084" rpy="0 0 0"/>
     <geometry>
       <mesh filename="package://vica_description/meshes/left_wheel_1.stl" scale="0.001 0.001 0.001"/>
@@ -65,5 +65,5 @@
   </inertial>
   <visual>
-    <origin xyz="-0.154 0.1465 0.084" rpy="0 0 0"/>
+    <origin xyz="-0.154 0.182 0.084" rpy="0 0 0"/>
     <geometry>
       <mesh filename="package://vica_description/meshes/right_wheel_1.stl" scale="0.001 0.001 0.001"/>
@@ -72,5 +72,5 @@
   </visual>
   <collision>
-    <origin xyz="-0.154 0.1465 0.084" rpy="0 0 0"/>
+    <origin xyz="-0.154 0.182 0.084" rpy="0 0 0"/>
     <geometry>
       <mesh filename="package://vica_description/meshes/right_wheel_1.stl" scale="0.001 0.001 0.001"/>
@@ -85,5 +85,5 @@
   </inertial>
   <visual>
-    <origin xyz="0.252 -0.0695 0.107" rpy="0 0 0"/>
+    <origin xyz="0.252 -0.0795 0.107" rpy="0 0 0"/>
     <geometry>
       <mesh filename="package://vica_description/meshes/front_left_caster_wheel_1.stl" scale="0.001 0.001 0.001"/>
@@ -92,5 +92,5 @@
   </visual>
   <collision>
-    <origin xyz="0.252 -0.0695 0.107" rpy="0 0 0"/>
+    <origin xyz="0.252 -0.0795 0.107" rpy="0 0 0"/>
     <geometry>
       <mesh filename="package://vica_description/meshes/front_left_caster_wheel_1.stl" scale="0.001 0.001 0.001"/>
@@ -105,5 +105,5 @@
   </inertial>
   <visual>
-    <origin xyz="0.252 0.0695 0.107" rpy="0 0 0"/>
+    <origin xyz="0.252 0.0795 0.107" rpy="0 0 0"/>
     <geometry>
       <mesh filename="package://vica_description/meshes/front_right_caster_wheel_1.stl" scale="0.001 0.001 0.001"/>
@@ -112,5 +112,5 @@
   </visual>
   <collision>
-    <origin xyz="0.252 0.0695 0.107" rpy="0 0 0"/>
+    <origin xyz="0.252 0.0795 0.107" rpy="0 0 0"/>
     <geometry>
       <mesh filename="package://vica_description/meshes/front_right_caster_wheel_1.stl" scale="0.001 0.001 0.001"/>
@@ -165,5 +165,5 @@
   </inertial>
   <visual>
-    <origin xyz="-0.185 -0.0 -0.236" rpy="0 0 0"/>
+    <origin xyz="-0.185 -0.0 -0.233" rpy="0 0 0"/>
     <geometry>
       <mesh filename="package://vica_description/meshes/lidar_1.stl" scale="0.001 0.001 0.001"/>
@@ -172,5 +172,5 @@
   </visual>
   <collision>
-    <origin xyz="-0.185 -0.0 -0.236" rpy="0 0 0"/>
+    <origin xyz="-0.185 -0.0 -0.233" rpy="0 0 0"/>
     <geometry>
       <mesh filename="package://vica_description/meshes/lidar_1.stl" scale="0.001 0.001 0.001"/>
@@ -189,5 +189,5 @@
 </link>
 <joint name="left_wheel_joint" type="continuous">
-  <origin xyz="0.154 0.1465 -0.125" rpy="0 0 0"/>
+  <origin xyz="0.154 0.182 -0.125" rpy="0 0 0"/>
   <parent link="base_link"/>
   <child link="left_wheel_1"/>
@@ -195,5 +195,5 @@
 </joint>
 <joint name="right_wheel_joint" type="continuous">
-  <origin xyz="0.154 -0.1465 -0.125" rpy="0 0 0"/>
+  <origin xyz="0.154 -0.182 -0.125" rpy="0 0 0"/>
   <parent link="base_link"/>
   <child link="right_wheel_1"/>
@@ -201,5 +201,5 @@
 </joint>
 <joint name="front_left_caster_wheel_joint" type="continuous">
-  <origin xyz="-0.03 -0.015 -0.0655" rpy="0 0 0"/>
+  <origin xyz="-0.03 -0.005 -0.0655" rpy="0 0 0"/>
   <parent link="front_left_caster_steer_1"/>
   <child link="front_left_caster_wheel_1"/>
@@ -207,5 +207,5 @@
 </joint>
 <joint name="front_right_caster_wheel_joint" type="continuous">
-  <origin xyz="-0.03 0.015 -0.0655" rpy="0 0 0"/>
+  <origin xyz="-0.03 0.005 -0.0655" rpy="0 0 0"/>
   <parent link="front_right_caster_steer_1"/>
   <child link="front_right_caster_wheel_1"/>

Commit message: refactor(urdf): 좌표 상수를 property로 묶는다
이번 오류 3건이 전부 손으로 적은 좌표 상수에서 나왔다. y 계열을 property 하나로
모으고 라이다 메시 z를 body_center_z 수식으로 바꿔, 같은 수를 두 번 적지 않게
한다. xacro 출력은 직전 커밋과 완전히 동일하다.

Co-Authored-By: Claude Opus 5 <noreply@anthropic.com>

File: src/vica_description/urdf/VICA.xacro (robot description, xacro)
@@ -12,4 +12,15 @@
 <xacro:property name="camera_y" value="0.0" />
 <xacro:property name="camera_z" value="0.130" />
+<!-- Drive wheel / caster geometry. Single source for every y coordinate. -->
+<!-- 줄자 실측(바퀴 중심 사이). CAD 0.3618과 2.2 mm 차이.
+     encoder.yaml의 wheel_base_m 0.37은 회전 시험으로 맞춘 오도메트리 보정 상수라
+     이 값과 다르다. 통일 대상이 아니다 — 스펙 3.1.1절. -->
+<xacro:property name="wheel_separation" value="0.364" />
+<xacro:property name="wheel_y" value="${wheel_separation / 2}" />
+<!-- CAD 실측: steer ±0.0845, wheel ±0.0795 -->
+<xacro:property name="caster_steer_y" value="0.0845" />
+<xacro:property name="caster_y" value="0.0795" />
+<!-- steer 링크 기준 wheel 조인트의 y. round()는 부동소수점 꼬리를 자른다. -->
+<xacro:property name="caster_wheel_dy" value="${round(caster_y - caster_steer_y, 6)}" />
 <link name="base_footprint"/>
 <joint name="base_footprint_joint" type="fixed">
@@ -45,5 +56,5 @@
   </inertial>
   <visual>
-    <origin xyz="-0.154 -0.182 0.084" rpy="0 0 0"/>
+    <origin xyz="-0.154 ${-wheel_y} 0.084" rpy="0 0 0"/>
     <geometry>
       <mesh filename="package://vica_description/meshes/left_wheel_1.stl" scale="0.001 0.001 0.001"/>
@@ -52,5 +63,5 @@
   </visual>
   <collision>
-    <origin xyz="-0.154 -0.182 0.084" rpy="0 0 0"/>
+    <origin xyz="-0.154 ${-wheel_y} 0.084" rpy="0 0 0"/>
     <geometry>
       <mesh filename="package://vica_description/meshes/left_wheel_1.stl" scale="0.001 0.001 0.001"/>
@@ -65,5 +76,5 @@
   </inertial>
   <visual>
-    <origin xyz="-0.154 0.182 0.084" rpy="0 0 0"/>
+    <origin xyz="-0.154 ${wheel_y} 0.084" rpy="0 0 0"/>
     <geometry>
       <mesh filename="package://vica_description/meshes/right_wheel_1.stl" scale="0.001 0.001 0.001"/>
@@ -72,5 +83,5 @@
   </visual>
   <collision>
-    <origin xyz="-0.154 0.182 0.084" rpy="0 0 0"/>
+    <origin xyz="-0.154 ${wheel_y} 0.084" rpy="0 0 0"/>
     <geometry>
       <mesh filename="package://vica_description/meshes/right_wheel_1.stl" scale="0.001 0.001 0.001"/>
@@ -85,5 +96,5 @@
   </inertial>
   <visual>
-    <origin xyz="0.252 -0.0795 0.107" rpy="0 0 0"/>
+    <origin xyz="0.252 ${-caster_y} 0.107" rpy="0 0 0"/>
     <geometry>
       <mesh filename="package://vica_description/meshes/front_left_caster_wheel_1.stl" scale="0.001 0.001 0.001"/>
@@ -92,5 +103,5 @@
   </visual>
   <collision>
-    <origin xyz="0.252 -0.0795 0.107" rpy="0 0 0"/>
+    <origin xyz="0.252 ${-caster_y} 0.107" rpy="0 0 0"/>
     <geometry>
       <mesh filename="package://vica_description/meshes/front_left_caster_wheel_1.stl" scale="0.001 0.001 0.001"/>
@@ -105,5 +116,5 @@
   </inertial>
   <visual>
-    <origin xyz="0.252 0.0795 0.107" rpy="0 0 0"/>
+    <origin xyz="0.252 ${caster_y} 0.107" rpy="0 0 0"/>
     <geometry>
       <mesh filename="package://vica_description/meshes/front_right_caster_wheel_1.stl" scale="0.001 0.001 0.001"/>
@@ -112,5 +123,5 @@
   </visual>
   <collision>
-    <origin xyz="0.252 0.0795 0.107" rpy="0 0 0"/>
+    <origin xyz="0.252 ${caster_y} 0.107" rpy="0 0 0"/>
     <geometry>
       <mesh filename="package://vica_description/meshes/front_right_caster_wheel_1.stl" scale="0.001 0.001 0.001"/>
@@ -125,5 +136,5 @@
   </inertial>
   <visual>
-    <origin xyz="0.222 0.0845 0.0415" rpy="0 0 0"/>
+    <origin xyz="0.222 ${caster_steer_y} 0.0415" rpy="0 0 0"/>
     <geometry>
       <mesh filename="package://vica_description/meshes/front_right_caster_steer_1.stl" scale="0.001 0.001 0.001"/>
@@ -132,5 +143,5 @@
   </visual>
   <collision>
-    <origin xyz="0.222 0.0845 0.0415" rpy="0 0 0"/>
+    <origin xyz="0.222 ${caster_steer_y} 0.0415" rpy="0 0 0"/>
     <geometry>
       <mesh filename="package://vica_description/meshes/front_right_caster_steer_1.stl" scale="0.001 0.001 0.001"/>
@@ -145,5 +156,5 @@
   </inertial>
   <visual>
-    <origin xyz="0.222 -0.0845 0.0415" rpy="0 0 0"/>
+    <origin xyz="0.222 ${-caster_steer_y} 0.0415" rpy="0 0 0"/>
     <geometry>
       <mesh filename="package://vica_description/meshes/front_left_caster_steer_1.stl" scale="0.001 0.001 0.001"/>
@@ -152,5 +163,5 @@
   </visual>
   <collision>
-    <origin xyz="0.222 -0.0845 0.0415" rpy="0 0 0"/>
+    <origin xyz="0.222 ${-caster_steer_y} 0.0415" rpy="0 0 0"/>
     <geometry>
       <mesh filename="package://vica_description/meshes/front_left_caster_steer_1.stl" scale="0.001 0.001 0.001"/>
@@ -165,5 +176,5 @@
   </inertial>
   <visual>
-    <origin xyz="-0.185 -0.0 -0.233" rpy="0 0 0"/>
+    <origin xyz="-0.185 -0.0 ${-(laser_z + body_center_z)}" rpy="0 0 0"/>
     <geometry>
       <mesh filename="package://vica_description/meshes/lidar_1.stl" scale="0.001 0.001 0.001"/>
@@ -172,5 +183,5 @@
   </visual>
   <collision>
-    <origin xyz="-0.185 -0.0 -0.233" rpy="0 0 0"/>
+    <origin xyz="-0.185 -0.0 ${-(laser_z + body_center_z)}" rpy="0 0 0"/>
     <geometry>
       <mesh filename="package://vica_description/meshes/lidar_1.stl" scale="0.001 0.001 0.001"/>
@@ -189,5 +200,5 @@
 </link>
 <joint name="left_wheel_joint" type="continuous">
-  <origin xyz="0.154 0.182 -0.125" rpy="0 0 0"/>
+  <origin xyz="0.154 ${wheel_y} -0.125" rpy="0 0 0"/>
   <parent link="base_link"/>
   <child link="left_wheel_1"/>
@@ -195,5 +206,5 @@
 </joint>
 <joint name="right_wheel_joint" type="continuous">
-  <origin xyz="0.154 -0.182 -0.125" rpy="0 0 0"/>
+  <origin xyz="0.154 ${-wheel_y} -0.125" rpy="0 0 0"/>
   <parent link="base_link"/>
   <child link="right_wheel_1"/>
@@ -201,5 +212,5 @@
 </joint>
 <joint name="front_left_caster_wheel_joint" type="continuous">
-  <origin xyz="-0.03 -0.005 -0.0655" rpy="0 0 0"/>
+  <origin xyz="-0.03 ${caster_wheel_dy} -0.0655" rpy="0 0 0"/>
   <parent link="front_left_caster_steer_1"/>
   <child link="front_left_caster_wheel_1"/>
@@ -207,5 +218,5 @@
 </joint>
 <joint name="front_right_caster_wheel_joint" type="continuous">
-  <origin xyz="-0.03 0.005 -0.0655" rpy="0 0 0"/>
+  <origin xyz="-0.03 ${-caster_wheel_dy} -0.0655" rpy="0 0 0"/>
   <parent link="front_right_caster_steer_1"/>
   <child link="front_right_caster_wheel_1"/>
@@ -213,5 +224,5 @@
 </joint>
 <joint name="front_right_caster_steer_joint" type="continuous">
-  <origin xyz="-0.222 -0.0845 -0.0825" rpy="0 0 0"/>
+  <origin xyz="-0.222 ${-caster_steer_y} -0.0825" rpy="0 0 0"/>
   <parent link="base_link"/>
   <child link="front_right_caster_steer_1"/>
@@ -219,5 +230,5 @@
 </joint>
 <joint name="front_left_caster_steer_joint" type="continuous">
-  <origin xyz="-0.222 0.0845 -0.0825" rpy="0 0 0"/>
+  <origin xyz="-0.222 ${caster_steer_y} -0.0825" rpy="0 0 0"/>
   <parent link="base_link"/>
   <child link="front_left_caster_steer_1"/>

Commit message: feat(urdf): camera_optical_frame을 추가한다
실물은 RealSense 드라이버가 optical 프레임을 발행하지만 Isaac에는 드라이버가
없다. 정본을 하나로 유지하려고 URDF가 제공한다. RealSense 기본 이름
(camera_color_optical_frame 등)은 TF 중복 충돌을 피하려고 쓰지 않는다.

Co-Authored-By: Claude Opus 5 <noreply@anthropic.com>

File: src/vica_description/urdf/VICA.xacro (robot description, xacro)
@@ -246,3 +246,12 @@
   <child link="camera_link"/>
 </joint>
+<!-- REP-103: +Z forward, +X right, +Y down -->
+<!-- 실물은 RealSense 드라이버가 자체 발행하지만, Isaac에는 드라이버가 없어
+     URDF가 제공해야 한다. 정본을 하나로 유지하려고 여기에 둔다. -->
+<link name="camera_optical_frame"/>
+<joint name="camera_optical_joint" type="fixed">
+  <origin xyz="0 0 0" rpy="-${pi/2} 0 -${pi/2}"/>
+  <parent link="camera_link"/>
+  <child  link="camera_optical_frame"/>
+</joint>
 </robot>

Commit message: feat(urdf): 카메라를 핸들 기둥 마스트로 옮긴다 (설계값 - 실측 대기)
camera_x 0.28683 -> -0.225, camera_z 0.130 -> 0.885 (지면 1.075 m).
2026-08-17 실주행에서 카메라를 높이니 주행이 좋아진 것을 확인하고
하드웨어 설계를 바꾸는 중이다.

STL 실측(base_link.stl)으로 자기 몸 가림을 계산했다:
  앞쪽 최고 구조물 0.385 m (x 0.1~0.3)
  카메라(-0.225, 1.075)에서의 내림각 52.5도, 시야 반각 32.3도
  -> 수평~아래 20도까지 자기 몸이 화면에 안 들어온다
  -> 아래 15도 권장 (바닥 사각 앞끝 1.17 -> 0.46 m). rpy 주석에 기록

IMU 어댑터는 안 바꾼다 - TF 의 회전만 쓰고(translation 무시) 각속도는
강체 어디서 재도 같다. EKF 도 vyaw 하나만 융합한다.

** 이 브랜치는 하드웨어가 실제로 이설된 뒤에만 주행에 쓴다. 옛 위치에
카메라가 달린 채 이 URDF 로 주행하면 깊이가 75 cm 어긋난 높이로 투영되어
바닥이 허리 높이 벽으로 지도에 들어간다. 이설 전 주행은 dev 로 한다. **

장착 후 지면->렌즈 중심 실측으로 두 값을 확정한다.

Co-Authored-By: Claude Opus 5 (1M context) <noreply@anthropic.com>

File: src/vica_description/urdf/VICA.xacro (robot description, xacro)
@@ -12,7 +12,17 @@
 <xacro:property name="laser_y" value="0.0" />
 <xacro:property name="laser_z" value="0.192" />
-<xacro:property name="camera_x" value="0.28683" />
+<!-- 2026-08-18 카메라 마스트 이설(설계값 — 실측 대기).
+     핸들 기둥 위, 지면에서 렌즈 중심 1075 mm, 몸통 뒤끝(-305)에서 앞으로 80 mm.
+       camera_x  0.28683 -> -0.225   (뒤로 51.2 cm)
+       camera_z  0.130   ->  0.885   (지면 1.075 - base_link 0.190. 위로 75.5 cm)
+     장착 후 지면->렌즈 중심을 줄자로 실측해 이 두 값을 확정한다.
+     footprint 때 도면과 실측이 달랐다(손잡이 29->19 cm).
+     기울여 달면 camera_joint 의 rpy 도 함께 바꾼다(아래 주석).
+     ** 이 값은 하드웨어가 실제로 이설된 뒤에만 유효하다. 옛 위치(앞 0.287/0.320)에
+     카메라가 달린 채 이 URDF 로 주행하면 nvblox 가 깊이를 75 cm 어긋난 높이로
+     투영한다. 이설 전 주행은 이 브랜치(feat/camera-mast)가 아니라 dev 로 한다. -->
+<xacro:property name="camera_x" value="-0.225" />
 <xacro:property name="camera_y" value="0.0" />
-<xacro:property name="camera_z" value="0.130" />
+<xacro:property name="camera_z" value="0.885" />
 <!-- Drive wheel / caster geometry. Single source for every y coordinate. -->
 <!-- 줄자 실측(바퀴 중심 사이). CAD 0.3618과 2.2 mm 차이.
@@ -244,4 +254,11 @@
   <child link="laser_frame"/>
 </joint>
+<!-- 마스트 장착 기울기. 지금은 수평(rpy 0 0 0)으로 둔다.
+     아래로 기울여 달면 pitch(가운데 값)만 바꾼다. URDF 는 pitch 양수 = 아래.
+       아래 15도(권장): rpy="0 0.262 0"  바닥 사각 앞끝 1.17 -> 0.46 m,
+                        0.35 m 앞 사람의 허벅지~가슴이 화면에 들어온다
+       아래 20도(한계): 앞쪽 0.385 m 구조물(x 0.1~0.3, STL 실측)이 화면
+                        하단에 걸리기 시작한다. 이 위로 기울이지 말 것.
+     기울기를 바꿔도 IMU 어댑터 파라미터는 안 바꾼다 - TF 회전을 자동으로 읽는다. -->
 <joint name="camera_joint" type="fixed">
   <origin xyz="${camera_x} ${camera_y} ${camera_z}" rpy="0 0 0"/>

Commit message: feat(urdf): 마스트·손잡이 바 미리보기 형상을 얹는다 (시각화 전용)
연장 기둥(0.863->1.075)·손잡이 바(지면 약 1.05, 카메라 7.5cm 뒤)·마운트 팔.
collision 에는 넣지 않는다 - footprint·계약 시험의 실측 기준(base_link.stl)을
지킨다. 치수는 어림값이며 실물 CAD 가 나오면 메시로 교체한다.

Co-Authored-By: Claude Opus 5 (1M context) <noreply@anthropic.com>

File: src/vica_description/urdf/VICA.xacro (robot description, xacro)
@@ -55,4 +55,28 @@
     <material name="body_blue"/>
   </visual>
+  <!-- 2026-08-18 마스트 재설계 미리보기 - **시각화 전용**. collision 에는 넣지
+       않는다(footprint·계약 시험의 실측 기준은 base_link.stl 그대로다).
+       기존 기둥(STL 안, 최고점 지면 0.863)을 카메라 높이(지면 1.075)까지
+       연장하고 손잡이 바를 카메라 바로 뒤에 붙인 새 설계의 어림 형상이다.
+       실물 CAD 가 나오면 이 프리미티브들을 새 메시로 교체한다.
+       좌표는 base_link 기준(지면 = 값 + 0.190). -->
+  <visual>
+    <!-- 연장 기둥: 기존 기둥 꼭대기(0.673)에서 카메라 높이(0.885)까지 -->
+    <origin xyz="-0.30 0 0.779" rpy="0 0 0"/>
+    <geometry><box size="0.05 0.05 0.212"/></geometry>
+    <material name="body_blue"/>
+  </visual>
+  <visual>
+    <!-- 손잡이 바: 카메라(x -0.225) 바로 뒤, 카메라 높이 부근(지면 약 1.05) -->
+    <origin xyz="-0.30 0 0.86" rpy="${pi/2} 0 0"/>
+    <geometry><cylinder radius="0.016" length="0.32"/></geometry>
+    <material name="body_blue"/>
+  </visual>
+  <visual>
+    <!-- 카메라 마운트 팔: 기둥에서 카메라 장착점(-0.225, 0.885)까지 -->
+    <origin xyz="-0.263 0 0.885" rpy="0 0 0"/>
+    <geometry><box size="0.075 0.04 0.03"/></geometry>
+    <material name="body_blue"/>
+  </visual>
   <collision>
     <origin xyz="0 0 -${body_center_z}" rpy="0 0 0"/>

Commit message: fix(urdf): 마스트 미리보기를 실제 손잡이 형상 연장으로 바꾼다
어림 프리미티브 3개(사용자 판정: 별로)를 지우고, base_link.stl 사본에서
지면 0.5 m 위 정점만 +212 mm 올린 base_link_mast_preview.stl 로 교체한다.
그 높이 위에는 기둥·손잡이뿐이라 손잡이 형태·방향은 그대로 두고 기둥
길이만 늘어난다. 손잡이 꼭대기 0.863 -> 1.075 m (카메라 높이).

visual 만 바꾼다. collision 은 base_link.stl 원본 그대로 - footprint·계약
시험의 실측 기준이다.

Co-Authored-By: Claude Opus 5 (1M context) <noreply@anthropic.com>

File: src/vica_description/urdf/VICA.xacro (robot description, xacro)
@@ -48,33 +48,16 @@
     <inertia ixx="2.402108" iyy="3.622523" izz="4.166828" ixy="0.0" iyz="-0.0" ixz="0.343284"/>
   </inertial>
+  <!-- 2026-08-18 마스트 미리보기 - **visual 만** 교체한다.
+       base_link_mast_preview.stl 은 base_link.stl 의 사본에서 지면 0.5 m 위
+       정점만 +212 mm 올린 것이다. 그 높이 위에는 기둥·손잡이뿐이라(실측:
+       다른 부위 최고 0.385 m) 손잡이 형태는 그대로 두고 기둥 길이만 늘어난다.
+       손잡이 꼭대기 0.863 -> 1.075 m (카메라 높이).
+       collision 은 base_link.stl 원본 그대로다 - footprint·계약 시험의 실측
+       기준이라 건드리지 않는다. 실물 CAD 가 나오면 이 메시를 교체한다. -->
   <visual>
     <origin xyz="0 0 -${body_center_z}" rpy="0 0 0"/>
     <geometry>
-      <mesh filename="package://vica_description/meshes/base_link.stl" scale="0.001 0.001 0.001"/>
-    </geometry>
-    <material name="body_blue"/>
-  </visual>
-  <!-- 2026-08-18 마스트 재설계 미리보기 - **시각화 전용**. collision 에는 넣지
-       않는다(footprint·계약 시험의 실측 기준은 base_link.stl 그대로다).
-       기존 기둥(STL 안, 최고점 지면 0.863)을 카메라 높이(지면 1.075)까지
-       연장하고 손잡이 바를 카메라 바로 뒤에 붙인 새 설계의 어림 형상이다.
-       실물 CAD 가 나오면 이 프리미티브들을 새 메시로 교체한다.
-       좌표는 base_link 기준(지면 = 값 + 0.190). -->
-  <visual>
-    <!-- 연장 기둥: 기존 기둥 꼭대기(0.673)에서 카메라 높이(0.885)까지 -->
-    <origin xyz="-0.30 0 0.779" rpy="0 0 0"/>
-    <geometry><box size="0.05 0.05 0.212"/></geometry>
-    <material name="body_blue"/>
-  </visual>
-  <visual>
-    <!-- 손잡이 바: 카메라(x -0.225) 바로 뒤, 카메라 높이 부근(지면 약 1.05) -->
-    <origin xyz="-0.30 0 0.86" rpy="${pi/2} 0 0"/>
-    <geometry><cylinder radius="0.016" length="0.32"/></geometry>
-    <material name="body_blue"/>
-  </visual>
-  <visual>
-    <!-- 카메라 마운트 팔: 기둥에서 카메라 장착점(-0.225, 0.885)까지 -->
-    <origin xyz="-0.263 0 0.885" rpy="0 0 0"/>
-    <geometry><box size="0.075 0.04 0.03"/></geometry>
+      <mesh filename="package://vica_description/meshes/base_link_mast_preview.stl" scale="0.001 0.001 0.001"/>
+    </geometry>
     <material name="body_blue"/>
   </visual>

Commit message: chore(urdf): 마스트 메시를 정식 이름으로 승격한다
base_link_mast_preview.stl -> base_link_mast.stl. 사용자가 이 형상을 새
설계의 정식 모델로 확정했다. visual 참조·주석을 함께 갱신한다.
collision 은 base_link.stl 원본 유지 - 실물 완성 후 재실측 전에는 바꾸지
않는다.

Co-Authored-By: Claude Opus 5 (1M context) <noreply@anthropic.com>

File: src/vica_description/urdf/VICA.xacro (robot description, xacro)
@@ -48,15 +48,16 @@
     <inertia ixx="2.402108" iyy="3.622523" izz="4.166828" ixy="0.0" iyz="-0.0" ixz="0.343284"/>
   </inertial>
-  <!-- 2026-08-18 마스트 미리보기 - **visual 만** 교체한다.
-       base_link_mast_preview.stl 은 base_link.stl 의 사본에서 지면 0.5 m 위
-       정점만 +212 mm 올린 것이다. 그 높이 위에는 기둥·손잡이뿐이라(실측:
-       다른 부위 최고 0.385 m) 손잡이 형태는 그대로 두고 기둥 길이만 늘어난다.
-       손잡이 꼭대기 0.863 -> 1.075 m (카메라 높이).
+  <!-- 2026-08-18 마스트 재설계 형상 - **visual 만** 교체한다(사용자 확정).
+       base_link_mast.stl 은 base_link.stl 을 이렇게 가공한 것이다:
+         - 뒤끝 전폭 레일(0.248~0.363)과 치마 삭제
+         - 손잡이 기둥을 카메라 상자 뒤면(-0.238)에 밀착, 밑동은 차체 안까지
+         - 그립은 형태 그대로 지면 1.045~1.075 (카메라 높이)
        collision 은 base_link.stl 원본 그대로다 - footprint·계약 시험의 실측
-       기준이라 건드리지 않는다. 실물 CAD 가 나오면 이 메시를 교체한다. -->
+       기준이라 실물 완성 후 재실측 전에는 바꾸지 않는다.
+       실물 CAD 가 나오면 이 메시를 교체한다. -->
   <visual>
     <origin xyz="0 0 -${body_center_z}" rpy="0 0 0"/>
     <geometry>
-      <mesh filename="package://vica_description/meshes/base_link_mast_preview.stl" scale="0.001 0.001 0.001"/>
+      <mesh filename="package://vica_description/meshes/base_link_mast.stl" scale="0.001 0.001 0.001"/>
     </geometry>
     <material name="body_blue"/>
