Commit message: fix(description): 카메라 높이를 줄자 실측 0.910 m 로 맞춘다
2026-08-18 에 넣은 1075 mm 는 설계값이었고 한 번도 재본 적이 없었다. 이번
재부착으로 실제 높이가 바뀌어, 바닥에서 카메라 몸체 중앙까지 910 mm 로
실측했다. D455 는 렌즈가 몸체 중앙 높이에 일렬이라 몸체 중앙 = 렌즈 중심이다.

  camera_z  0.885 -> 0.720   (지면 0.910 - base_link 0.190. 16.5 cm 내려감)

오차 방향이 비대칭이라 그냥 두면 안 된다. URDF 가 실물보다 높으면 nvblox 가
바닥을 그만큼 띄워 투영해 slice 띠(0.05~0.9) 한가운데에 걸리고 주변이 통째로
장애물이 된다. 반대로 낮으면 바닥·사람이 띠 아래로 꺼져 nvblox 가 조용히 꺼진
것처럼 된다(2026-08-17 에 겪었다).

rpy 는 0 0 0 을 유지한다. D455 내장 IMU 로 재니 roll +0.24도, pitch +0.49도로
4 m 앞 3.5 cm 수준이라 넣을 값이 없다.

visual 메시(base_link_mast.stl)는 옛 1.075 기준 그대로 둔다. RViz 에서 카메라가
마스트 그립보다 16.5 cm 아래에 그려지지만 메시는 TF·footprint·nvblox 어디에도
안 물린다. 그 사실을 주석에 남겼다.

검증: tf2_echo base_footprint camera_link -> [-0.225, 0.000, 0.910], rpy 0 0 0

Co-Authored-By: Claude Opus 5 (1M context) <noreply@anthropic.com>

File: src/vica_description/urdf/VICA.xacro (robot description, xacro)
@@ -12,17 +12,23 @@
 <xacro:property name="laser_y" value="0.0" />
 <xacro:property name="laser_z" value="0.192" />
-<!-- 2026-08-18 카메라 마스트 이설(설계값 — 실측 대기).
-     핸들 기둥 위, 지면에서 렌즈 중심 1075 mm, 몸통 뒤끝(-305)에서 앞으로 80 mm.
-       camera_x  0.28683 -> -0.225   (뒤로 51.2 cm)
-       camera_z  0.130   ->  0.885   (지면 1.075 - base_link 0.190. 위로 75.5 cm)
-     장착 후 지면->렌즈 중심을 줄자로 실측해 이 두 값을 확정한다.
-     footprint 때 도면과 실측이 달랐다(손잡이 29->19 cm).
-     기울여 달면 camera_joint 의 rpy 도 함께 바꾼다(아래 주석).
-     ** 이 값은 하드웨어가 실제로 이설된 뒤에만 유효하다. 옛 위치(앞 0.287/0.320)에
-     카메라가 달린 채 이 URDF 로 주행하면 nvblox 가 깊이를 75 cm 어긋난 높이로
-     투영한다. 이설 전 주행은 이 브랜치(feat/camera-mast)가 아니라 dev 로 한다. -->
+<!-- 2026-08-24 줄자 실측으로 확정. 앞서 있던 1075 mm 는 2026-08-18 이설 때 넣은
+     설계값이었고 한 번도 재본 적이 없었다. 이번 재부착으로 실제 높이가 바뀌었다.
+     바닥에서 카메라 몸체 중앙까지 실측 910 mm (D455 는 렌즈가 몸체 중앙 높이에
+     일렬로 놓여 몸체 중앙 = 렌즈 중심이다).
+       camera_x  -0.225          (몸통 뒤끝 -305 에서 앞으로 80 mm. 이번에 그대로)
+       camera_z   0.885 -> 0.720 (지면 0.910 - base_link 0.190. 16.5 cm 내려감)
+     rpy 는 0 0 0 이 맞다 - D455 내장 IMU 로 재니 roll +0.24도, pitch +0.49도로
+     4 m 앞 3.5 cm 수준이라 넣을 값이 없다(2026-08-24).
+     ** 높이가 실물과 어긋나면 nvblox 가 깊이를 그만큼 어긋난 높이로 투영한다.
+     오차 방향이 비대칭이다. URDF 가 실물보다 **높으면** 바닥이 떠올라 slice
+     띠(0.05~0.9)에 걸려 주변이 통째로 장애물이 되고, **낮으면** 바닥·사람이 띠
+     아래로 꺼져 nvblox 가 조용히 꺼진 것처럼 된다(2026-08-17 에 실제로 겪었다).
+     카메라를 다시 달 때마다 줄자로 재서 이 값을 고친다.
+     ** visual 메시(base_link_mast.stl)는 옛 1.075 기준 그대로다(2026-08-24 사용자 판단).
+     RViz 에서 카메라가 마스트 그립보다 16.5 cm 아래에 그려지는데 정상이다. 메시는
+     TF·footprint·nvblox 어디에도 안 물린다 - 화면 그림일 뿐이다. -->
 <xacro:property name="camera_x" value="-0.225" />
 <xacro:property name="camera_y" value="0.0" />
-<xacro:property name="camera_z" value="0.885" />
+<xacro:property name="camera_z" value="0.720" />
 <!-- Drive wheel / caster geometry. Single source for every y coordinate. -->
 <!-- 줄자 실측(바퀴 중심 사이). CAD 0.3618과 2.2 mm 차이.

Commit message: fix(description): 카메라 높이를 재고정 실측 1.05 m 로 맞춘다
재부착으로 0.910 -> 1.050 m (사용자 고정). depth 바닥 실측으로 검증:
광선각 20.6/26.6/29.4도에서 높이차 1.05/1.03/1.04 m 일정 = 높이·수평 일치.
camera_z 0.720 -> 0.860. 재학습 데이터셋(robot_view_dataset)도 이 높이에서
촬영됨(CAPTURE_INFO.md).

Co-Authored-By: Claude Fable 5 <noreply@anthropic.com>
Claude-Session: https://claude.ai/code/session_01SBWJs3nzeAJhrX24pyNb8i

File: src/vica_description/urdf/VICA.xacro (robot description, xacro)
@@ -30,5 +30,7 @@
 <xacro:property name="camera_x" value="-0.225" />
 <xacro:property name="camera_y" value="0.0" />
-<xacro:property name="camera_z" value="0.720" />
+<!-- 2026-08-25 재고정: 지면 1.05 m (사용자 고정 + depth 바닥 실측 1.03~1.05 로 확인).
+     camera_z = 1.05 - base_link 0.190 = 0.860. 수평(rpy 0 0 0)도 같은 실측으로 유지 확인. -->
+<xacro:property name="camera_z" value="0.860" />
 <!-- Drive wheel / caster geometry. Single source for every y coordinate. -->
 <!-- 줄자 실측(바퀴 중심 사이). CAD 0.3618과 2.2 mm 차이.

Commit message: fix(description,nav2): 카메라 높이와 차체 세로 실측을 반영한다
2026-08-29 줄자 실측(사용자 확정)으로 두 값이 바뀌었다.

- camera_z 0.860 -> 0.835. 지면 1.05 -> 1.025 m 다. nvblox 가 깊이를 투영하는
  높이라 실물과 어긋나면 바닥이 뜨거나(주변이 통째로 장애물) 꺼진다(조용히
  안 보임). 2026-08-17 에 실제로 겪은 실패라 1 cm 도 넘기지 않는다.
- footprint 후방 -0.495 -> -0.415. 손잡이 돌출이 19 -> 11 cm 로 줄어 총 세로가
  80 -> 72 cm 가 됐다. 앞(+0.305)과 반폭(±0.225)은 그대로다. local·global
  두 costmap 에 같은 값을 넣는다.

내접반경은 0.275 m 로 바뀌지 않는다. 내접은 가장 가까운 변까지의 거리이고 그
변은 차체 좌우 변이라 뒤를 줄여도 움직이지 않는다. 그래서 통과 가능성 판정과
inflation_radius 0.56 은 손대지 않았다. 줄어든 것은 외접반경뿐이다.

  외접  0.5516 -> 0.4727 m   제자리 회전 직경 1.10 -> 0.95 m

inflation 0.56 이 옛 외접 0.5516 을 덮었으므로 새 값은 더 넉넉히 덮는다.
test_footprint_contract 의 MEASURED_REAR 를 함께 갱신했다. 계약 시험 33개 통과,
xacro 파싱과 colcon build 확인.

실주행 미검증이다.

Co-Authored-By: Claude Opus 5 (1M context) <noreply@anthropic.com>
Claude-Session: https://claude.ai/code/session_01AepQieuYGsA2SsFz95nDTC

File: src/vica_description/urdf/VICA.xacro (robot description, xacro)
@@ -30,7 +30,10 @@
 <xacro:property name="camera_x" value="-0.225" />
 <xacro:property name="camera_y" value="0.0" />
-<!-- 2026-08-25 재고정: 지면 1.05 m (사용자 고정 + depth 바닥 실측 1.03~1.05 로 확인).
-     camera_z = 1.05 - base_link 0.190 = 0.860. 수평(rpy 0 0 0)도 같은 실측으로 유지 확인. -->
-<xacro:property name="camera_z" value="0.860" />
+<!-- 2026-08-29 재고정: 지면 1.025 m (줄자 실측, 사용자 확정).
+     camera_z = 1.025 - base_link 0.190 = 0.835. 2026-08-25 값(지면 1.05 / 0.860)에서
+     2.5 cm 내려왔다. 같은 회차에 차체 세로가 80 -> 72 cm 로 줄었지만 그쪽은 이 값과
+     무관하다 - nav2_params.yaml 의 footprint 후방(-0.495 -> -0.415)이 받는다.
+     수평(rpy 0 0 0)은 이번에 바꾸지 않았다. -->
+<xacro:property name="camera_z" value="0.835" />
 <!-- Drive wheel / caster geometry. Single source for every y coordinate. -->
 <!-- 줄자 실측(바퀴 중심 사이). CAD 0.3618과 2.2 mm 차이.

Commit message: feat(nav2,description): D455 깊이를 2D 스캔으로 눌러 costmap 에 넣고 마스트 기울기 3도를 실측 반영한다
라이다는 지면 0.382 m 단일 평면만 본다. 그 밖의 물체 -- 책상 상판·다리 -- 는
어떤 costmap 에도 안 들어와 8/29 주행에서 "방 -> 경유지2 / 입구"가 두 번
충돌로 막혔다. 깊이를 두 번째 눈으로 넣는다.

## 1. 마스트가 위로 3.0도 들려 있었다 (VICA.xacro)

URDF 는 수평(rpy 0 0 0)이라고 알고 있었다. 그 어긋남 때문에 바닥점이 20~40 cm
떠서 계산됐고, costmap 이 로봇 앞을 통째로 LETHAL 로 덮어 "길이 막혔다"가 났다.
3도는 2 m 앞에서 10.5 cm 다.

  재는 법  깊이 포인트클라우드에서 바닥 평면을 RANSAC 으로 찾아 법선의 앞뒤
           성분을 읽는다(평면 두께 9 mm, 점 9,000개). 앞에 물건이 있어도 견딘다.
  실측     3.05 / 2.88 / 3.16 / 3.06 도 -> 3.04 +- 0.14
  부호     측정기의 양수는 "URDF 보다 위로 들렸다" 이므로 URDF pitch 에는
           뒤집어 넣는다. 처음 +0.0524 를 넣었더니 오차가 3 -> 6.3도로 두 배가
           되어 확정했다.

같은 측정에서 카메라 높이는 1.008 m 로 나왔다(URDF 1.025 와 1.7 cm 차이).
줄자 실측의 오차 범위라 camera_z 는 건드리지 않는다.

이 수정은 카메라를 쓰는 모든 기능(사람 검출, 나중에 되살릴 nvblox)에 함께 듣는다.

## 2. 깊이는 3D 가 아니라 2D 로 넣는다 (nav2_params.yaml, launch)

처음에는 포인트클라우드를 그대로 voxel_layer 에 넣었다. 책상 다리는 잘 봤지만
**찍은 칸을 지우지 못했다.** bag 실측(run2017, 846초, 4,714칸):

  0.9~1.8 m (깊이가 찍는 구간)   3,833칸   수명 중앙 21.6초   최대 191초
  1.8 m 밖  (라이다 구간)           451칸   수명 중앙  0.6초
  방향별: 정면·좌우 24~26초 / 뒤쪽(라이다만) 0.6~1.2초
  로봇 상태별: 정지 22.2초 / 주행 12.6초  ← 안 움직이면 더 안 지워진다

원인은 카메라 높이다. 지면 1.025 m 에서 그보다 낮은 칸을 지우려면 그 칸을
스치는 광선이 훨씬 먼 바닥까지 닿아야 한다.

  R = d / (1 - h / 1.025)
  d 1.8 · h 0.60 -> 4.3 m    d 1.8 · h 0.75 -> 6.7 m    d 1.8 · h 0.90 -> 9.8 m

실내는 3~4 m 앞에 벽이 있어 그만한 바닥이 안 보인다. raytrace_max_range 를
8 m 로 늘려도 볼 바닥이 없으면 소용이 없었다(전반 28.7 -> 후반 10.2초에서 멈춤).
라이다가 잘 지워지는 이유는 **자기와 같은 높이를 보기 때문**이다.

그래서 깊이도 한 평면으로 누른다. 0.30~1.05 m 띠의 점을 LaserScan 으로 바꿔
넣으면 마킹도 청소도 같은 평면에서 일어난다.

  pointcloud_to_laserscan  target_frame base_footprint, 띠 0.30~1.05 m,
                           +-43도 173빔, range 0.30~4.0 m, use_inf
  costmap depth_scan       높이 창 -0.05~0.15(지면 층), 표시 0.3~3.0 m,
                           persistence 0.0, expected_update_rate 0.0

높이 창 아래끝을 0.0 이 아니라 -0.05 로 둔다. nav2 는 관측점을 odom 으로 옮긴
뒤 `pz < min_obstacle_height` 로 거르는데 스캔이 정확히 z=0 이라 경계에 걸린다.
0.0 일 때 스캔은 빔의 95 %에 물체를 잡는데 costmap 은 0~4칸이었다.

라이다(0.382 m 층)와 다른 층을 쓰므로 서로의 마크를 지우지 않는다. z_voxels 는
2D 가 된 뒤 높은 격자가 불필요해져 24 -> 16 으로 되돌렸다.

잃는 것은 높이 정보다. 테이블 상판이 잡히면 그 아래가 뚫려 있어도 막힌 것으로
보지만, 이 로봇은 손잡이 때문에 어차피 못 지나간다.

## 3. 계약 시험 13개 (test_depth_voxel_contract.py)

오늘 세 번 같은 함정에 빠져서 규칙으로 박는다.
  - data_type 이 LaserScan 인가 (PointCloud2 로 되돌리면 유령이 재발한다)
  - 스캔을 만드는 쪽(launch)과 받는 쪽(costmap)의 값이 맞물리는가
  - 높이 띠 아래끝이 흔들림을 견디는가 / 위끝이 로봇 최고점 이하인가
  - URDF 의 camera_z·camera_pitch 가 이 계산과 일치하는가
  - 라이다와 다른 층을 쓰는가

## 미검증

정지 상태에서 사람이 코앞(0.44 m)에 섰다 비킨 뒤 그 자리가 20초 내내 0칸으로
남는 것은 확인했다. **비킨 순간을 기준으로 한 정확한 소거 시간은 아직 못 쟀다.**
실주행 검증도 남았다. 되돌리려면 marking 을 끄면 된다(재기동 불필요):
  ros2 param set /local_costmap/local_costmap voxel_layer.depth_scan.marking false

Co-Authored-By: Claude Opus 5 (1M context) <noreply@anthropic.com>
Claude-Session: https://claude.ai/code/session_01LgxjnNVygiQMkLUSgcc3LS

File: src/vica_description/urdf/VICA.xacro (robot description, xacro)
@@ -36,4 +36,19 @@
      수평(rpy 0 0 0)은 이번에 바꾸지 않았다. -->
 <xacro:property name="camera_z" value="0.835" />
+<!-- 2026-08-29 저녁 실측: 마스트가 위로 3.0도 들려 있다(pitch 음수).
+     재는 법 - 깊이 포인트클라우드에서 바닥 평면을 RANSAC 으로 찾아
+     그 법선의 앞뒤 성분을 읽었다(평면 두께 9 mm, 점 9,000개).
+     4회 측정 3.05 / 2.88 / 3.16 / 3.06 도 -> 3.04 +- 0.14.
+     부호 주의: 이 측정기가 내는 양수는 "URDF 가 믿는 자세보다 위로 들렸다"는
+     뜻이라 URDF pitch 에는 부호를 뒤집어 넣는다. 처음에 +0.0524 를 넣었더니
+     오차가 3도에서 6.3도로 두 배가 되어 부호를 확정했다(같은 날 실측).
+     같은 측정에서 카메라 높이는 1.008 m 로 나왔다. URDF 의 1.025 와
+     1.7 cm 차이인데 줄자 실측의 오차 범위라 camera_z 는 건드리지 않는다.
+     왜 이 값이 필요한가: URDF 가 수평이라고 믿는 동안 바닥점이 20~40 cm
+     떠서 계산됐고, local_costmap 의 깊이 소스가 그것을 통째로 장애물로
+     찍어 로봇 앞이 까맣게 찼다("길이 막혔다"). 3도는 2 m 앞에서 10.5 cm 다.
+     카메라를 물리적으로 수평에 맞추는 대신 실제 각도를 여기 적는다 -
+     기울어져 있어도 TF 가 알기만 하면 계산은 정확해진다. -->
+<xacro:property name="camera_pitch" value="-0.0524" />  <!-- 3.0 도, 위로 -->
 <!-- Drive wheel / caster geometry. Single source for every y coordinate. -->
 <!-- 줄자 실측(바퀴 중심 사이). CAD 0.3618과 2.2 mm 차이.
@@ -273,6 +288,10 @@
   <child link="laser_frame"/>
 </joint>
-<!-- 마스트 장착 기울기. 지금은 수평(rpy 0 0 0)으로 둔다.
-     아래로 기울여 달면 pitch(가운데 값)만 바꾼다. URDF 는 pitch 양수 = 아래.
+<!-- 마스트 장착 기울기. 2026-08-29 실측으로 위 3.0도(camera_pitch)를 넣었다.
+     이 값은 "이렇게 달자"는 설계값이 아니라 "실제로 이렇게 달려 있다"는 실측값이다.
+     마스트를 손대면 반드시 다시 재서 이 값을 고쳐야 한다. 안 고치면 바닥이
+     장애물로 찍혀 앞이 막힌다(2026-08-29 실주행에서 겪음).
+     재는 도구: 바닥 평면 RANSAC. 절차는 camera_pitch 선언부 주석 참조.
+     아래로 더 기울여 달면 pitch(가운데 값)만 바꾼다. URDF 는 pitch 양수 = 아래.
        아래 15도(권장): rpy="0 0.262 0"  바닥 사각 앞끝 1.17 -> 0.46 m,
                         0.35 m 앞 사람의 허벅지~가슴이 화면에 들어온다
@@ -281,5 +300,5 @@
      기울기를 바꿔도 IMU 어댑터 파라미터는 안 바꾼다 - TF 회전을 자동으로 읽는다. -->
 <joint name="camera_joint" type="fixed">
-  <origin xyz="${camera_x} ${camera_y} ${camera_z}" rpy="0 0 0"/>
+  <origin xyz="${camera_x} ${camera_y} ${camera_z}" rpy="0 ${camera_pitch} 0"/>
   <parent link="base_link"/>
   <child link="camera_link"/>

Commit message: fix(description): 카메라 재장착 후 높이·기울기를 다시 실측해 반영한다
카메라를 탈착 후 재장착하면서 자세가 바뀌었다.

  높이     1.025 -> 1.045 m   (지면에서 렌즈 중심까지, 줄자 실측)
           camera_z 0.835 -> 0.855
  기울기   위로 3.00도 -> 위로 0.71도
           camera_pitch -0.0524 -> -0.0124

기울기 측정 3회 -2.35 / -2.31 / -2.24 도, 편차 0.05. 평면 두께 8 mm, 점 17,000개.
바닥 평면 RANSAC 으로 쟀다(scripts/vica_camera_pitch.py).

## 도구의 결함을 하나 고쳤다

이 도구가 재는 것은 **URDF 기준 잔여 오차**다. TF 가 이미 camera_pitch 를 반영하고
있기 때문이다. 따라서 새 값은 절대값이 아니라

    새 값 = 지금 값 + 잔여 오차를 되돌리는 양

인데, 도구가 절대값을 찍어 주고 있었다. 이번에 그대로 넣었다면 -3.00 도에
+2.30 도를 넣어 오차가 오히려 커졌을 것이다. 2026-08-29 에 부호를 뒤집어 넣어
오차가 두 배가 됐던 것과 같은 종류의 함정이다.

도구가 URDF 를 직접 읽어 계산하도록 고쳤다. 계약 시험 상수는 URDF 와 **같은 부호**
(음수 = 위로)이므로 그것도 뒤집지 않도록 함께 바로잡았다.

Co-Authored-By: Claude Opus 5 (1M context) <noreply@anthropic.com>
Claude-Session: https://claude.ai/code/session_01LgxjnNVygiQMkLUSgcc3LS

File: src/vica_description/urdf/VICA.xacro (robot description, xacro)
@@ -34,6 +34,10 @@
      2.5 cm 내려왔다. 같은 회차에 차체 세로가 80 -> 72 cm 로 줄었지만 그쪽은 이 값과
      무관하다 - nav2_params.yaml 의 footprint 후방(-0.495 -> -0.415)이 받는다.
-     수평(rpy 0 0 0)은 이번에 바꾸지 않았다. -->
-<xacro:property name="camera_z" value="0.835" />
+     수평(rpy 0 0 0)은 이번에 바꾸지 않았다.
+     2026-08-30 재고정: 지면 1.045 m (줄자 실측, 사용자 확정).
+     camera_z = 1.045 - base_link 0.190 = 0.855. 카메라를 탈착 후 재장착하면서
+     2.0 cm 올라갔다. **탈부착할 때마다 높이와 기울기를 함께 재는 것을 절차로
+     삼는다** - 아래 camera_pitch 주석의 도구가 둘을 같이 출력한다. -->
+<xacro:property name="camera_z" value="0.855" />
 <!-- 2026-08-29 저녁 실측: 마스트가 위로 3.0도 들려 있다(pitch 음수).
      재는 법 - 깊이 포인트클라우드에서 바닥 평면을 RANSAC 으로 찾아
@@ -50,5 +54,14 @@
      카메라를 물리적으로 수평에 맞추는 대신 실제 각도를 여기 적는다 -
      기울어져 있어도 TF 가 알기만 하면 계산은 정확해진다. -->
-<xacro:property name="camera_pitch" value="-0.0524" />  <!-- 3.0 도, 위로 -->
+<xacro:property name="camera_pitch" value="-0.0124" />  <!-- 0.7 도, 위로 -->
+<!-- 2026-08-30 재장착 후 재측정: 3.0도 -> 0.7도 (둘 다 위로).
+     같은 회차에 높이도 1.025 -> 1.045 m 로 2 cm 올라갔다(줄자 실측).
+     이 도구가 재는 것은 **URDF 기준 잔여 오차**다. TF 가 이미 camera_pitch 를
+     반영하고 있기 때문이다. 따라서 새 값은 절대값이 아니라
+         새 값 = 지금 값 + 잔여 오차를 되돌리는 양
+     이다. 이번에 -3.00 도에서 잔여 -2.29 도가 나왔으므로 -0.71 도가 됐다.
+     도구가 이 계산을 대신하도록 고쳤다(scripts/vica_camera_pitch.py).
+     그 전에는 절대값을 찍어 줘서, 그대로 넣으면 오차가 오히려 커졌다.
+     측정 3회 -2.35 / -2.31 / -2.24 도, 편차 0.05. 평면 두께 8 mm, 점 17,000개. -->
 <!-- Drive wheel / caster geometry. Single source for every y coordinate. -->
 <!-- 줄자 실측(바퀴 중심 사이). CAD 0.3618과 2.2 mm 차이.

Commit message: feat(nav2,description): 초음파 URDF 링크와 센서별 range 레이어를 단다
- VICA.xacro: usonic_front_left/right 링크 (+0.305, ±0.107, -0.0987, 수평).
  드라이버 ultrasonic_frame_ids 와 이름 일치 필수
- local_costmap: range_sensor_front_left/right 두 레이어로 분리해서 추가.
  한 레이어에 두 토픽을 넣으면 확률 장부를 공유해, 겹침 구역에서 비스듬한
  면에 소리가 튕긴 센서의 거짓 '에코 없음'이 이웃 센서의 마크까지 지운다
  — 실주행에서 LETHAL 109->0->109 깜빡임으로 로봇이 상자를 밀고 갔다.
  분리하면 clear 는 자기 장부만 지우고 master 는 max 결합이라 마크가
  남는다. 장애물이 정말 사라지면 양쪽 다 지워 잔상도 안 남는다
- clear_on_max_reading true(부채꼴 청소), no_readings_timeout 0.0(보조
  센서 fail-open — 초음파가 죽어도 주행을 멈추지 않는다)
- global_costmap 미적용: 방위 분해능이 없어 저장 지도를 뭉갠다

실기: 한쪽 센서가 10초간 clear 를 읽어도 반대쪽 마크 유지·cmd 0 —
정지 유지 실증(usonic_drive04·08 bag). 조기 감지 1.0~1.2m -> 점진 감속.
계약 시험 76개 통과(기존 dev 실패 2건은 본 변경과 무관).

Co-Authored-By: Claude Fable 5 <noreply@anthropic.com>
Claude-Session: https://claude.ai/code/session_01Nr4RVBupFvpBqJZQQdqEaw

File: src/vica_description/urdf/VICA.xacro (robot description, xacro)
@@ -12,4 +12,13 @@
 <xacro:property name="laser_y" value="0.0" />
 <xacro:property name="laser_z" value="0.192" />
+<!-- 초음파 DYP-A22 x2 (2026-08-31): 앞범퍼 중앙에서 좌우 107mm, 지면 91.3mm,
+     수평 장착(틸트 불가 확정). docs/handoff_jetson_ultrasonic_i2c.md §6.6.
+     frame 이름은 드라이버 ultrasonic_frame_ids 와 일치해야 한다.
+     z = 0.0913(지면) - 0.190(base_link) = -0.0987.
+     [실측 확인] 센서가 범퍼 앞면(+0.305)보다 튀어나와 있으면 usonic_x 와
+     footprint 앞단을 함께 키워야 한다(같은 문서 §6.6 주의). -->
+<xacro:property name="usonic_x" value="0.305" />
+<xacro:property name="usonic_y" value="0.107" />
+<xacro:property name="usonic_z" value="-0.0987" />
 <!-- 2026-08-24 줄자 실측으로 확정. 앞서 있던 1075 mm 는 2026-08-18 이설 때 넣은
      설계값이었고 한 번도 재본 적이 없었다. 이번 재부착으로 실제 높이가 바뀌었다.
@@ -301,4 +310,17 @@
   <child link="laser_frame"/>
 </joint>
+<!-- 초음파: 빔 축 = +x(전방), 수평. Range 메시지의 부채꼴이 이 frame 에서 그려진다. -->
+<link name="usonic_front_left"/>
+<joint name="usonic_front_left_joint" type="fixed">
+  <origin xyz="${usonic_x} ${usonic_y} ${usonic_z}" rpy="0 0 0"/>
+  <parent link="base_link"/>
+  <child link="usonic_front_left"/>
+</joint>
+<link name="usonic_front_right"/>
+<joint name="usonic_front_right_joint" type="fixed">
+  <origin xyz="${usonic_x} ${-usonic_y} ${usonic_z}" rpy="0 0 0"/>
+  <parent link="base_link"/>
+  <child link="usonic_front_right"/>
+</joint>
 <!-- 마스트 장착 기울기. 2026-08-29 실측으로 위 3.0도(camera_pitch)를 넣었다.
      이 값은 "이렇게 달자"는 설계값이 아니라 "실제로 이렇게 달려 있다"는 실측값이다.

Commit message: feat(description): 초음파 센서를 URDF 에 보이게 한다
usonic_front_left/right 가 visual 없는 빈 링크라 rviz 에서 TF 축만 떴다.
센서가 실제로 어디에 붙어 있는지, 범퍼 앞면보다 튀어나오지는 않는지를 눈으로
확인할 수 없었다.

DYP-A22 일반 규격(방수 원통형, 직경 22 mm · 길이 20 mm)을 cylinder 로 넣는다.
카메라(D455)를 box placeholder 로 둔 것과 같은 방식이다.

링크 원점은 **센서 앞면**(측정 원점)이고 몸체는 그 뒤로 뻗으므로, 원통 중심을
길이의 절반만큼 -x 로 물렸다. 이걸 빼먹으면 실물보다 20 mm 앞으로 튀어나온
것처럼 그려져 usonic_x(0.305)와 범퍼 앞면의 관계를 눈으로 읽을 때 틀리게 된다.

URDF cylinder 의 축은 z 라서 빔 축 +x 에 맞추려면 y 로 90도 눕힌다.

collision 은 넣지 않는다. 주행 충돌 판정은 nav2 footprint 가 하고 URDF
collision 은 거기에 관여하지 않는다. 시각 확인이 목적이므로 보이는 것만 둔다.

[미검증] 치수는 실물을 잰 값이 아니라 일반 규격이다(사용자 지정). 줄자로
확인하면 usonic_diameter / usonic_length 두 값만 고치면 된다.

xacro 전개 확인: radius 0.011 · length 0.02 · rpy "0 1.5708 0" · xyz "-0.01 0 0".

Co-Authored-By: Claude Opus 5 (1M context) <noreply@anthropic.com>
Claude-Session: https://claude.ai/code/session_01HwjMjHwLAKnGqHKgvGtgJp

File: src/vica_description/urdf/VICA.xacro (robot description, xacro)
@@ -310,6 +310,28 @@
   <child link="laser_frame"/>
 </joint>
-<!-- 초음파: 빔 축 = +x(전방), 수평. Range 메시지의 부채꼴이 이 frame 에서 그려진다. -->
-<link name="usonic_front_left"/>
+<!-- 초음파: 빔 축 = +x(전방), 수평. Range 메시지의 부채꼴이 이 frame 에서 그려진다.
+     visual 은 DYP-A22 일반 규격(방수 원통형)을 옮긴 것이다. 2026-09-02 추가.
+     [미검증] 실물을 재서 넣은 값이 아니다. 줄자로 확인하면 아래 두 값만 고친다.
+     링크 원점은 **센서 앞면**(측정 원점)이고 몸체는 그 뒤로 뻗는다. 그래서
+     원통 중심을 길이의 절반만큼 -x 로 물린다. 이걸 빼먹으면 실물보다 20 mm
+     앞으로 튀어나온 것처럼 그려져, 범퍼 앞면(usonic_x 0.305)과의 관계를 눈으로
+     확인할 때 잘못 읽게 된다.
+     URDF cylinder 의 축은 z 다. 빔 축 +x 에 맞추려면 y 로 90도 눕힌다.
+     collision 은 넣지 않는다. 주행 충돌 판정은 nav2 footprint 가 하고 URDF
+     collision 은 거기에 관여하지 않는다. 시각 확인이 목적이므로 보이는 것만 둔다. -->
+<xacro:property name="usonic_diameter" value="0.022" />
+<xacro:property name="usonic_length" value="0.020" />
+<xacro:macro name="usonic_visual">
+  <visual name="dyp_a22_body">
+    <origin xyz="${-usonic_length/2} 0 0" rpy="0 ${pi/2} 0"/>
+    <geometry>
+      <cylinder radius="${usonic_diameter/2}" length="${usonic_length}"/>
+    </geometry>
+    <material name="silver"/>
+  </visual>
+</xacro:macro>
+<link name="usonic_front_left">
+  <xacro:usonic_visual/>
+</link>
 <joint name="usonic_front_left_joint" type="fixed">
   <origin xyz="${usonic_x} ${usonic_y} ${usonic_z}" rpy="0 0 0"/>
@@ -317,5 +339,7 @@
   <child link="usonic_front_left"/>
 </joint>
-<link name="usonic_front_right"/>
+<link name="usonic_front_right">
+  <xacro:usonic_visual/>
+</link>
 <joint name="usonic_front_right_joint" type="fixed">
   <origin xyz="${usonic_x} ${-usonic_y} ${usonic_z}" rpy="0 0 0"/>
