Commit message: fix(description,nav2): base_link 원점을 차체 중심에서 구동륜 축으로 15.4 cm 옮긴다
차동구동이라 실제 회전 중심은 구동륜 축 중점이다. 그런데 base_link 원점은 CAD
원점인 차체 한가운데였고 구동륜 joint 가 거기서 x +0.154 에 있었다. 한편
encoder_feedback.py(292~299행)는 좌우 바퀴 이동거리의 평균과 차이로
odom -> base_footprint 를 내므로, TF 가 실제로 추적하는 점은 이미 구동륜 축이었다.
보정 항은 없다. 즉 '오도메트리가 가리키는 점'과 '거기 붙여 둔 몸 모양'이
15.4 cm 어긋난 채로 돌아가고 있었다.

nav2_params.yaml 의 footprint 주석은 "base_link(구동륜 축) 기준"이라고 적고 있었다.
전제는 처음부터 구동륜 축이었고 URDF 만 그것을 안 지켰다.

로봇은 설정과 무관하게 이미 구동륜 축으로 돈다. 이 커밋은 로봇을 바꾸는 것이
아니라 로봇이 자기 몸을 제대로 알게 하는 것이다.

무엇이 달라지나

  footprint x 범위     -0.415~+0.305  ->  -0.569~+0.151
  내접(padding 포함)    0.2750 m       ->  0.2010 m
  외접(padding 포함)    0.4727 m       ->  0.6248 m
  제자리 회전 필요 폭    0.945 m        ->  1.250 m

제자리 회전에서 뒤쪽이 실제로 쓸고 가던 15.4 cm 를 이제 검사한다. 180도 회전이면
차체 중앙이 실제로 0.308 m 움직이는데 그동안 제자리로 계산하고 있었다. 라이다도
실제로는 회전축에서 3.1 cm 앞인데 TF 는 18.5 cm 로 알아, 회전 중 라이다가 움직일
거리를 6배 크게 예측했다.

같이 옮긴 것 (하나라도 빠지면 지도·costmap 이 통째로 틀어진다)

  - VICA.xacro: axle_offset_x 신설. base_link 를 parent 로 하는 joint 8개와
    base_link 자신의 visual·collision·inertial origin. 줄자 실측값(laser_x 0.185 등)은
    그대로 두고 joint 에서 빼는 방식이라 다음 사람이 줄자와 대조할 수 있다.
    base_footprint 는 x 오프셋이 0 이라 함께 따라온다.
  - nav2_params.yaml: 두 costmap 의 footprint, collision_monitor 다각형 2개.
  - test_footprint_contract.py: 실측 기준은 차체 중심으로 두고 비교 직전에
    AXLE_OFFSET_X 를 뺀다. 내접반경을 Nav2 방식(padFootprint + 가장 가까운 변)으로
    직접 계산하게 고쳤다 - 원점이 옮겨지며 '반폭 + padding' 이 더 이상 내접이
    아니게 됐기 때문이다(이제 앞면이 더 가깝다). URDF 의 axle_offset_x 와 이 파일의
    상수가 어긋나면 멈추는 시험을 추가했다.
  - test_nav2_launch_contract.py: 차체 앞단 0.355 하드코딩을 footprint 계산으로 교체.
  - test_pose_score.py, pose_bootstrap_node.py: 낡은 주석 정정. 센서 오프셋은
    TF 에서 읽으므로 코드는 자동으로 따라간다.

[실패하는 시험 1개 — 고치지 않았다]

  test_planner_contract::test_turning_radius_clears_the_narrowest_measured_corner[active]

  격자 R 0.10 이 90도 코너에 요구하는 폭이 0.84 m 에서 1.10 m 로 늘었고,
  MEASURED_NARROWEST_CORRIDOR 도 1.10 이라 여유가 0 이 됐다. 이 상수는
  2026-07-30 옛 건물 줄자값이라 지금 장소에는 맞지 않는다. 통로 실측이
  이 시험을 판정한다. **느슨하게 고치지 말 것** - 이 시험이 알리는 신호가
  이번 변경의 핵심 결과다.

  나머지 실패 2개(nvblox_dependency, recovery_patience)는 이 변경 전에도 실패한다.

[미검증] 실기에서 회전 중심을 직접 재지는 않았다. 09-15 실주행에서 TF·costmap 이
새 값을 쓰는 것과, 1.4 m 통로에서 제자리 회전 비율이 47 % -> 77 % 로 오른 것은
확인했다. 줄자로 앞 범퍼 끝에서 구동축 중심까지를 재면 0.151 m 가 나와야 한다.

[관찰] 같은 날 bag 분석: planner 는 최소 곡률반경 0.100 m 경로를 제대로 그리는데
컨트롤러가 실행한 호는 중앙 0.21~0.26 m 였다(필요 폭 1.41~1.48 m). 1.2·1.3·1.4 m
통로에서 모두 못 빠져나온 것은 폭이 아니라 이 격차 때문이다. 별개 과제다.

Co-Authored-By: Claude Opus 5 <noreply@anthropic.com>
Claude-Session: https://claude.ai/code/session_01EhkWCwANw8dQQiwadQ2Es9

File: src/vica_description/urdf/VICA.xacro (robot description, xacro)
@@ -9,4 +9,34 @@
 <xacro:property name="body_center_z" value="0.041" />
 <xacro:property name="base_link_height" value="0.19" />
+<!-- ── 2026-09-15 base_link 원점을 차체 중심에서 구동륜 축으로 옮긴다 ──────────
+     이 로봇은 차동구동이라 **실제 회전 중심은 구동륜 축 중점**이다. 그런데
+     base_link 원점은 CAD 원점인 차체 한가운데였고, 구동륜 joint 가 거기서
+     x +0.154 에 있었다. 두 점이 15.4 cm 어긋나 있었다는 뜻이다.
+     왜 문제인가. encoder_feedback.py 는 좌우 바퀴 이동거리의 평균과 차이로
+     d_center·d_theta 를 구해 odom -> base_footprint 로 낸다(293~299행). 이
+     계산이 뜻하는 점은 교과서대로 **구동륜 축 중점**이고 보정 항은 없다.
+     그래서 'TF 가 실제로 추적하는 점'과 '거기 붙여 둔 몸 모양(footprint·
+     라이다·카메라 위치)'이 15.4 cm 어긋나 있었다.
+     결과로 나타나던 것:
+       - 제자리 회전 시 뒤쪽이 쓸고 가는 반경을 Nav2 가 0.154 m 짧게 봤다
+         (0.4727 -> 실제 0.6248, padding 포함). 코너에서 뒤가 스쳤다.
+       - 180도 제자리 회전이면 차체 중앙이 실제로 0.308 m 움직이는데
+         Nav2 는 제자리로 계산했다.
+       - 라이다는 실제 회전축에서 3.1 cm 앞인데 TF 는 18.5 cm 로 알아,
+         회전 중 라이다가 움직일 거리를 6배 크게 예측했다.
+     로봇은 설정과 무관하게 이미 구동륜 축으로 돈다. 이 수정은 로봇을 바꾸는
+     것이 아니라 로봇이 자기 몸을 제대로 알게 하는 것이다.
+     같이 움직여야 하는 것(하나라도 빠지면 지도·costmap 이 전부 틀어진다):
+       ① base_link 의 visual·collision·inertial origin  (이 파일)
+       ② base_link 를 parent 로 하는 joint 9개          (이 파일)
+       ③ nav2_params.yaml 의 footprint 2곳 · collision_monitor 다각형 2개
+       ④ test_footprint_contract.py 의 실측 기준 좌표
+     base_footprint 는 base_link 의 부모이고 x 오프셋이 0 이라 함께 따라온다.
+     이 값이 틀리면 전부 틀린다. 줄자로 **앞 범퍼 끝에서 구동축 중심까지**를
+     재면 0.305 - 0.154 = 0.151 m 가 나와야 한다. 다르면 여기만 고친다. -->
+<xacro:property name="axle_offset_x" value="0.154" />
+<!-- 아래 센서 x 값은 전부 **차체 중심** 기준 줄자 실측이다. base_link 원점은
+     이제 구동륜 축이므로 joint 에서 axle_offset_x 를 뺀다. 실측값 자체는
+     그대로 두어야 다음 사람이 줄자와 대조할 수 있다. -->
 <xacro:property name="laser_x" value="0.185" />
 <xacro:property name="laser_y" value="0.0" />
@@ -92,5 +122,5 @@
 <link name="base_link">
   <inertial>
-    <origin xyz="0.004031215194176557 3.002726997808124e-17 0.03506562657816282" rpy="0 0 0"/>
+    <origin xyz="${0.004031215194176557 - axle_offset_x} 3.002726997808124e-17 0.03506562657816282" rpy="0 0 0"/>
     <mass value="90.84709962539795"/>
     <inertia ixx="2.402108" iyy="3.622523" izz="4.166828" ixy="0.0" iyz="-0.0" ixz="0.343284"/>
@@ -105,5 +135,5 @@
        실물 CAD 가 나오면 이 메시를 교체한다. -->
   <visual>
-    <origin xyz="0 0 -${body_center_z}" rpy="0 0 0"/>
+    <origin xyz="${-axle_offset_x} 0 -${body_center_z}" rpy="0 0 0"/>
     <geometry>
       <mesh filename="package://vica_description/meshes/base_link_mast.stl" scale="0.001 0.001 0.001"/>
@@ -112,5 +142,5 @@
   </visual>
   <collision>
-    <origin xyz="0 0 -${body_center_z}" rpy="0 0 0"/>
+    <origin xyz="${-axle_offset_x} 0 -${body_center_z}" rpy="0 0 0"/>
     <geometry>
       <mesh filename="package://vica_description/meshes/base_link.stl" scale="0.001 0.001 0.001"/>
@@ -269,5 +299,5 @@
 </link>
 <joint name="left_wheel_joint" type="continuous">
-  <origin xyz="0.154 ${wheel_y} -0.125" rpy="0 0 0"/>
+  <origin xyz="${0.154 - axle_offset_x} ${wheel_y} -0.125" rpy="0 0 0"/>
   <parent link="base_link"/>
   <child link="left_wheel_1"/>
@@ -275,5 +305,5 @@
 </joint>
 <joint name="right_wheel_joint" type="continuous">
-  <origin xyz="0.154 ${-wheel_y} -0.125" rpy="0 0 0"/>
+  <origin xyz="${0.154 - axle_offset_x} ${-wheel_y} -0.125" rpy="0 0 0"/>
   <parent link="base_link"/>
   <child link="right_wheel_1"/>
@@ -293,5 +323,5 @@
 </joint>
 <joint name="front_right_caster_steer_joint" type="continuous">
-  <origin xyz="-0.222 ${-caster_steer_y} -0.0825" rpy="0 0 0"/>
+  <origin xyz="${-0.222 - axle_offset_x} ${-caster_steer_y} -0.0825" rpy="0 0 0"/>
   <parent link="base_link"/>
   <child link="front_right_caster_steer_1"/>
@@ -299,5 +329,5 @@
 </joint>
 <joint name="front_left_caster_steer_joint" type="continuous">
-  <origin xyz="-0.222 ${caster_steer_y} -0.0825" rpy="0 0 0"/>
+  <origin xyz="${-0.222 - axle_offset_x} ${caster_steer_y} -0.0825" rpy="0 0 0"/>
   <parent link="base_link"/>
   <child link="front_left_caster_steer_1"/>
@@ -306,5 +336,5 @@
 <!-- Sensor positions are expressed relative to the body-centered base_link. -->
 <joint name="laser_joint" type="fixed">
-  <origin xyz="${laser_x} ${laser_y} ${laser_z}" rpy="0 0 0"/>
+  <origin xyz="${laser_x - axle_offset_x} ${laser_y} ${laser_z}" rpy="0 0 0"/>
   <parent link="base_link"/>
   <child link="laser_frame"/>
@@ -335,5 +365,5 @@
 </link>
 <joint name="usonic_front_left_joint" type="fixed">
-  <origin xyz="${usonic_x} ${usonic_y} ${usonic_z}" rpy="0 0 0"/>
+  <origin xyz="${usonic_x - axle_offset_x} ${usonic_y} ${usonic_z}" rpy="0 0 0"/>
   <parent link="base_link"/>
   <child link="usonic_front_left"/>
@@ -343,5 +373,5 @@
 </link>
 <joint name="usonic_front_right_joint" type="fixed">
-  <origin xyz="${usonic_x} ${-usonic_y} ${usonic_z}" rpy="0 0 0"/>
+  <origin xyz="${usonic_x - axle_offset_x} ${-usonic_y} ${usonic_z}" rpy="0 0 0"/>
   <parent link="base_link"/>
   <child link="usonic_front_right"/>
@@ -359,5 +389,5 @@
      기울기를 바꿔도 IMU 어댑터 파라미터는 안 바꾼다 - TF 회전을 자동으로 읽는다. -->
 <joint name="camera_joint" type="fixed">
-  <origin xyz="${camera_x} ${camera_y} ${camera_z}" rpy="0 ${camera_pitch} 0"/>
+  <origin xyz="${camera_x - axle_offset_x} ${camera_y} ${camera_z}" rpy="0 ${camera_pitch} 0"/>
   <parent link="base_link"/>
   <child link="camera_link"/>

Commit message: feat(guidance,nav2,description): 초음파 8채널 — 펌웨어·파서·URDF·costmap 레이어
왜
- 09-22 에 센서 8개(0x68~0x6F)를 자리별로 실측했지만 펌웨어·ROS 는 앞 두 개만 읽었다.
  사용자 요청(09-23): 8개 전부 costmap 에 넣는다. 유효 거리·발행 fov 는 앞 두 개와 동일
  (1.5 m, 물리 빔 50°, 지도 표시 30°).

무엇을
- 펌웨어: 서로 등진 채널 2개를 한 라운드로 묶어 4라운드(420 ms/바퀴, 채널당 약 2.4 Hz).
  같은 방향 센서는 서로의 메아리를 읽으므로(인수인계 §4.2) 절대 같이 쏘지 않는다.
  상향에 8채널 프레임 AA 57(20 B) 추가. 옛 AA 55(8 B, 앞 두 개)는 라운드 B 뒤에 호환용으로
  계속 보낸다 — 옛 파서 워크스페이스에서도 앞 두 채널이 보이게. US_SEND_LEGACY 로 끈다.
- protocol/ultrasonic_frame: 헤더 AA 57·20 B·8채널로 일반화. 옛 프레임은 헤더가 달라 무시.
  시험 12개(레거시 무시·자리 순서 포함), 터치 혼합 시험 갱신. 130 통과.
- user_guidance.yaml: 토픽·frame_id·measurement_delay 8개(자리 번호 순, 라운드별 지연).
- VICA.xacro: 초음파 링크 6개 추가(usonic_link 매크로, yaw 로 방향). 좌표는 차체 치수에서
  추정한 값 [미검증] — RViz 대조·줄자 실측 뒤 고칠 것.
- nav2_params: local costmap 에 range_sensor_* 8개(센서별 분리, 08-31 확정 방식), 전부
  enabled True (09-16 False 는 초음파 미연결 회차용이었다). 설정은 여덟 레이어 동일.

검증: 파서·설정 pytest 130 통과 / xacro 전개·check_urdf 성공 / nav2 config 시험은
수정 전후 동일(기존 실패 3건 외 신규 없음) / 펌웨어 컴파일 통과. 실기 미검증.

Co-Authored-By: Claude Fable 5.1 <noreply@anthropic.com>

File: src/vica_description/urdf/VICA.xacro (robot description, xacro)
@@ -377,4 +377,34 @@
   <child link="usonic_front_right"/>
 </joint>
+<!-- ── 2026-09-23 초음파 6개 추가 → 8개 배치 (자리↔주소 실측표: devlog/2026-09-22-esp32-스마트핸들-이식.md) ──
+     아래 x/y 는 줄자 실측이 **아니라 차체 치수(footprint 주석)에서 추정한 값**이다 [미검증].
+     기준은 앞 센서와 같은 차체 중심이고, joint 에서 axle_offset_x 를 뺀다.
+       바퀴 옆(1·4번)      x = +0.154 (구동륜 축)          y = ±0.225 (차체 반폭)
+       뒷바퀴 옆(8·5번)    x = -0.252 (앞 캐스터 x 의 대칭 가정) y = ±0.225
+       후방(7·6번)         x = -0.305 (차체 뒷면)          y = ±0.107 (앞 센서와 같은 간격 가정)
+       높이는 전부 앞 센서와 같다고 가정(usonic_z).
+     yaw 는 센서가 보는 방향: 왼쪽 +90° / 오른쪽 -90° / 후방 180°. 부채꼴(Range)은 이
+     방향으로 그려지므로, RViz 에서 실물과 어긋나면 **줄자로 재서 이 값들을 고친다.**
+     link 이름은 user_guidance.yaml 의 ultrasonic_frame_ids 와 반드시 일치해야 한다. -->
+<xacro:property name="usonic_side_x"       value="0.154" />
+<xacro:property name="usonic_side_y"       value="0.225" />
+<xacro:property name="usonic_rear_wheel_x" value="-0.252" />
+<xacro:property name="usonic_rear_x"       value="-0.305" />
+<xacro:macro name="usonic_link" params="name x y yaw">
+  <link name="${name}">
+    <xacro:usonic_visual/>
+  </link>
+  <joint name="${name}_joint" type="fixed">
+    <origin xyz="${x - axle_offset_x} ${y} ${usonic_z}" rpy="0 0 ${yaw}"/>
+    <parent link="base_link"/>
+    <child link="${name}"/>
+  </joint>
+</xacro:macro>
+<xacro:usonic_link name="usonic_left_wheel"       x="${usonic_side_x}"       y="${usonic_side_y}"  yaw="${pi/2}"/>   <!-- 1번 -->
+<xacro:usonic_link name="usonic_right_wheel"      x="${usonic_side_x}"       y="${-usonic_side_y}" yaw="${-pi/2}"/>  <!-- 4번 -->
+<xacro:usonic_link name="usonic_right_rear_wheel" x="${usonic_rear_wheel_x}" y="${-usonic_side_y}" yaw="${-pi/2}"/>  <!-- 5번 -->
+<xacro:usonic_link name="usonic_rear_right"       x="${usonic_rear_x}"       y="${-usonic_y}"      yaw="${pi}"/>     <!-- 6번 -->
+<xacro:usonic_link name="usonic_rear_left"        x="${usonic_rear_x}"       y="${usonic_y}"       yaw="${pi}"/>     <!-- 7번 -->
+<xacro:usonic_link name="usonic_left_rear_wheel"  x="${usonic_rear_wheel_x}" y="${usonic_side_y}"  yaw="${pi/2}"/>   <!-- 8번 -->
 <!-- 마스트 장착 기울기. 2026-08-29 실측으로 위 3.0도(camera_pitch)를 넣었다.
      이 값은 "이렇게 달자"는 설계값이 아니라 "실제로 이렇게 달려 있다"는 실측값이다.
